Commit message: Separación Controladores
Se separaron los controladores y se crearon dos robots con 2 descripciones distintas

File: ProyectoInt/urdf/phantom2_description_gazebo.xacro (robot description, xacro)
@@ -1,14 +1,14 @@
 <?xml version="1.0" ?>
-<robot name="phantom" xmlns:xacro="http://www.ros.org/wiki/xacro">
+<robot name="phantom2" xmlns:xacro="http://www.ros.org/wiki/xacro">
   <xacro:include filename="$(find ProyectoInt)/urdf/links_joints.xacro" />
   <xacro:include filename="$(find ProyectoInt)/urdf/robot_parameters.xacro" />
-  <link name="world">
+  <link name="world2">
   </link>
-  <joint name="joint_name" type="fixed">
-    <parent link="world"/>
-    <child link="${link_00_name}"/>
+  <joint name="joint_name2" type="fixed">
+    <parent link="world2"/>
+    <child link="${link_00_name2}"/>
     <origin xyz="0.0 0.0 0.0" rpy="0.0 0.0 0.0"/>
   </joint>
-  <xacro:m_link_mesh name="${link_00_name}"
+  <xacro:m_link_mesh name="${link_00_name2}"
     origin_xyz="0 0 0"
     origin_rpy="0 0 0"
@@ -19,12 +19,12 @@
     izz="0.000704614"
   />
-  <xacro:m_joint name="${joint_01_name}"
+  <xacro:m_joint name="${joint_01_name2}"
     type="revolute"
     axis_xyz="0 0 1"
     origin_rpy="0 0 0" origin_xyz="0 0 0"
-    parent="${link_00_name}" child="${link_01_name}"
+    parent="${link_00_name2}" child="${link_01_name2}"
     limit_e="100" limit_l="-3.14" limit_u="3.14" limit_v="0.5"
   />
-  <xacro:m_link_mesh name="${link_01_name}"
+  <xacro:m_link_mesh name="${link_01_name2}"
     origin_xyz="0 0 0.095"
     origin_rpy="0 0 0"
@@ -35,12 +35,12 @@
     izz="0.000018984"
   />
-  <xacro:m_joint name="${joint_02_name}"
+  <xacro:m_joint name="${joint_02_name2}"
     type="revolute"
     axis_xyz="0 0 1"
     origin_rpy="-1.57 0 0" origin_xyz="0 0 0.137"
-    parent="${link_01_name}" child="${link_02_name}"
+    parent="${link_01_name2}" child="${link_02_name2}"
     limit_e="100" limit_l="-3.14" limit_u="3.14" limit_v="0.5"
   />
-  <xacro:m_link_mesh name="${link_02_name}"
+  <xacro:m_link_mesh name="${link_02_name2}"
     origin_xyz="0 0 0"
     origin_rpy="1.57 0 1.57"
@@ -51,12 +51,12 @@
     izz="0.000031204"
   />
-  <xacro:m_joint name="${joint_03_name}"
+  <xacro:m_joint name="${joint_03_name2}"
     type="revolute"
     axis_xyz="0 0 1"
     origin_rpy="0 0 0" origin_xyz="0.105 0 0"
-    parent="${link_02_name}" child="${link_03_name}"
+    parent="${link_02_name2}" child="${link_03_name2}"
     limit_e="100" limit_l="-3.14" limit_u="3.14" limit_v="0.5"
   />
-  <xacro:m_link_mesh name="${link_03_name}"
+  <xacro:m_link_mesh name="${link_03_name2}"
     origin_xyz="0 0 0"
     origin_rpy="1.57 0 1.57"
@@ -67,12 +67,12 @@
     izz="0.000031204"
   />
-  <xacro:m_joint name="${joint_04_name}"
+  <xacro:m_joint name="${joint_04_name2}"
     type="revolute"
     axis_xyz="0 0 1"
     origin_rpy="0 0 0" origin_xyz="0.105 0 0"
-    parent="${link_03_name}" child="${link_04_name}"
+    parent="${link_03_name2}" child="${link_04_name2}"
     limit_e="100" limit_l="-3.14" limit_u="3.14" limit_v="0.5"
   />
-  <xacro:m_link_mesh name="${link_04_name}"
+  <xacro:m_link_mesh name="${link_04_name2}"
     origin_xyz="0 0 0"
     origin_rpy="1.57 0 1.57"
@@ -83,12 +83,12 @@
     izz="0.000053899"
   />
-  <xacro:m_joint name="${joint_05_name}"
+  <xacro:m_joint name="${joint_05_name2}"
     type="prismatic"
     axis_xyz="0 0 1"
     origin_rpy="0 0 0" origin_xyz="0.071 0 -0.03"
-    parent="${link_04_name}" child="${link_05_name}"
+    parent="${link_04_name2}" child="${link_05_name2}"
     limit_e="100" limit_l="0" limit_u="0.016" limit_v="0.5"
   />
-  <xacro:m_link_mesh name="${link_05_name}"
+  <xacro:m_link_mesh name="${link_05_name2}"
     origin_xyz="0 0 0"
     origin_rpy="1.57 0 1.57"
@@ -99,13 +99,13 @@
     izz="0.000002959"
   />
-  <xacro:m_joint_mimic name="${joint_06_name}"
+  <xacro:m_joint_mimic name="${joint_06_name2}"
     type="prismatic"
     axis_xyz="0 0 1"
     origin_rpy="3.14 0 0" origin_xyz="0.071 0 0.03"
-    parent="${link_04_name}" child="${link_06_name}"
+    parent="${link_04_name2}" child="${link_06_name2}"
     limit_e="100" limit_l="0" limit_u="0.016" limit_v="0.5"
-    mimic_joint="${joint_05_name}" m_multiplier="1" m_offset="0"
+    mimic_joint="${joint_05_name2}" m_multiplier="1" m_offset="0"
   />
-  <xacro:m_link_mesh name="${link_06_name}"
+  <xacro:m_link_mesh name="${link_06_name2}"
     origin_xyz="0 0 0"
     origin_rpy="1.57 0 1.57"
@@ -119,5 +119,5 @@
     origin_xyz="0.11 0 0"
     origin_rpy="-1.57 0 -1.57"
-    parent="${link_04_name}"
+    parent="${link_04_name2}"
   />
   <gazebo>

File: ProyectoInt/urdf/robot_parameters.xacro (robot description, xacro)
@@ -14,3 +14,16 @@
   <xacro:property name="joint_05_name" value="gripper_1" />
   <xacro:property name="joint_06_name" value="gripper_2" />
+  <xacro:property name="link_00_name2" value="robot_base2" />
+  <xacro:property name="link_01_name2" value="link2_01" />
+  <xacro:property name="link_02_name2" value="link2_02" />
+  <xacro:property name="link_03_name2" value="link2_03" />
+  <xacro:property name="link_04_name2" value="link2_04" />
+  <xacro:property name="link_05_name2" value="finger2_1" />
+  <xacro:property name="link_06_name2" value="finger2_2" />
+  <xacro:property name="joint_01_name2" value="joint2_1" />
+  <xacro:property name="joint_02_name2" value="joint2_2" />
+  <xacro:property name="joint_03_name2" value="joint2_3" />
+  <xacro:property name="joint_04_name2" value="joint2_4" />
+  <xacro:property name="joint_05_name2" value="gripper2_1" />
+  <xacro:property name="joint_06_name2" value="gripper2_2" />
 </robot>
