Commit message: Escalando zona de trabajo

File: ProyectoInt/urdf/zona_alimentacion.xacro (robot description, xacro)
@@ -4,6 +4,6 @@
         <inertial>
           <origin xyz="0.0 0.0 0.0" rpy="0.0 0.0 0.0" />
-          <mass value="6.365" />
-          <inertia  ixx="0.026003677" ixy="0.0"  ixz="0.0"  iyy="0.137391177"  iyz="0.0"  izz="0.153820833" />
+          <mass value="0.353" />
+          <inertia  ixx="0.000518226" ixy="0.0"  ixz="0.0"  iyy="0.000682845"  iyz="0.0"  izz="0.001158212" />
         </inertial>
         <visual>

File: ProyectoInt/urdf/zona_ensamble.xacro (robot description, xacro)
@@ -4,6 +4,6 @@
         <inertial>
           <origin xyz="0.0 0.0 0.0" rpy="0.0 0.0 0.0" />
-          <mass value="1.790" />
-          <inertia  ixx="0.004590694" ixy="0.0"  ixz="-0.001181006"  iyy="0.009780904"  iyz="0.0"  izz="0.011903296" />
+          <mass value="0.882" />
+          <inertia  ixx="0.001438432" ixy="0.0"  ixz="-0.000330708"  iyy="0.004406841"  iyz="0.0"  izz="0.005452392" />
         </inertial>
         <visual>

Commit message: Zonas fijas
Se fijaron las zonas de alimentación y ensamble al suelo. Además se dejo el script de pick and place del primer robot para que fuese más parámetrico.

File: ProyectoInt/urdf/zona_alimentacion.xacro (robot description, xacro)
@@ -1,4 +1,11 @@
 <?xml version="1.0"?>
 <robot name="Zona_Alimentacion">
+      <link name="world">
+      </link>
+      <joint name="joint_name" type="fixed">
+        <parent link="world"/>
+        <child link="alimentacion"/>
+        <origin xyz="0.0 0.0 0.0" rpy="0.0 0.0 0.0"/>
+      </joint>
       <link name="alimentacion">
         <inertial>

File: ProyectoInt/urdf/zona_ensamble.xacro (robot description, xacro)
@@ -1,4 +1,11 @@
 <?xml version="1.0"?>
 <robot name="Zona_Ensamble">
+      <link name="world">
+      </link>
+      <joint name="joint_name" type="fixed">
+        <parent link="world"/>
+        <child link="ensamble"/>
+        <origin xyz="0.0 0.0 0.0" rpy="0.0 0.0 0.0"/>
+      </joint>
       <link name="ensamble">
         <inertial>
